Commit message: material tags added in urdf

File: explore_bot/urdf/camera.xacro (robot description, xacro)
@@ -21,5 +21,5 @@
     <link name="camera_link_optical"></link>
     <gazebo reference="camera_link">
-        <material>Gazebo/Red</material>
+        <material>Gazebo/Black</material>
         <sensor name="camera" type="camera">
             <pose> 0 0 0 0 0 0 </pose>

File: explore_bot/urdf/robot.urdf.xacro (robot description, xacro)
@@ -4,4 +4,5 @@
     <xacro:include filename="gazebo_control.xacro"/>
     <xacro:include filename="camera.xacro" />
+    <xacro:include filename="robot.gazebo"/>
     <material name="white">
         <color rgba="1 1 1 1" />
@@ -11,5 +12,5 @@
     </material>
     <material name="blue">
-        <color rgba="0.2 0.2 1 1"/>
+        <color rgba="0.203125 0.23828125 0.28515625 1.0"/>
     </material>
     <material name="black">
@@ -31,5 +32,5 @@
                 <box size="0.3 0.3 0.15"/>
             </geometry>
-            <material name="white"/>
+            <material name="red"/>
         </visual>
         <collision>
@@ -43,4 +44,7 @@
         </xacro:inertial_box>
     </link>
+    <!-- <gazebo reference="chassis">
+        <material>Gazebo/Red</material>
+    </gazebo> -->
     <!-- LEFT WHEEL LINK -->
     <joint name="left_wheel_joint" type="continuous">
@@ -55,5 +59,5 @@
                 <cylinder radius="0.05" length="0.04"/>
             </geometry>
-            <material name="blue"/>
+            <material name="white"/>
         </visual>
         <collision>
@@ -78,5 +82,5 @@
                 <cylinder radius="0.05" length="0.04"/>
             </geometry>
-            <material name="blue"/>
+            <material name="white"/>
         </visual>
         <collision>
