Commit message: robot base inertia updated

File: explore_bot/urdf/inertial_macros.xacro (robot description, xacro)
@@ -8,13 +8,4 @@
                     iyy="${(2/5) * mass * (radius*radius)}" iyz="0.0"
                     izz="${(2/5) * mass * (radius*radius)}" />
-        </inertial>
-    </xacro:macro>
-    <xacro:macro name="inertial_box" params="mass x y z *origin">
-        <inertial>
-            <xacro:insert_block name="origin"/>
-            <mass value="${mass}" />
-            <inertia ixx="${(1/12) * mass * (y*y+z*z)}" ixy="0.0" ixz="0.0"
-                    iyy="${(1/12) * mass * (x*x+z*z)}" iyz="0.0"
-                    izz="${(1/12) * mass * (x*x+y*y)}" />
         </inertial>
     </xacro:macro>

File: explore_bot/urdf/robot.urdf.xacro (robot description, xacro)
@@ -40,11 +40,6 @@
             </geometry>
         </collision>
-        <xacro:inertial_box mass="0.5" x="0.3" y="0.3" z="0.15">
-            <origin xyz="0.15 0 0.075" rpy="0 0 0"/>
-        </xacro:inertial_box>
+        <inertia ixx="0.0395416666667" ixy="0" ixz="0" iyy="0.106208333333" iyz="0" izz="0.106208333333"/>
     </link>
-    <!-- <gazebo reference="chassis">
-        <material>Gazebo/Red</material>
-    </gazebo> -->
     <!-- LEFT WHEEL LINK -->
     <joint name="left_wheel_joint" type="continuous">
